Commit message: first try at debugging self collision

File: experiments/assets/ur5/ur5.urdf (robot description, URDF)
Before this commit: robot ur5, 13 links, 12 joints
Links:
- link ee_link: geometry 
- link wrist_3_link: geometry visual mesh filename=visual/wrist3.stl

Commit message: simplified collision meshes to cylinders

File: experiments/assets/ur5/ur5.urdf (robot description, URDF)
Before this commit: robot ur5, 13 links, 12 joints
Links:
- link base_link: geometry visual mesh filename=visual/base.stl
- link ee_link: geometry 
- link forearm_link: geometry collision cylinder length=0.4 radius=0.04; visual mesh filename=visual/forearm.stl
- link shoulder_link: geometry collision cylinder length=0.2 radius=0.05; visual mesh filename=visual/shoulder.stl
- link upper_arm_link: geometry collision cylinder length=0.4 radius=0.05; visual mesh filename=visual/upperarm.stl
- link wrist_1_link: geometry collision cylinder length=0.1 radius=0.035; visual mesh filename=visual/wrist1.stl
- link wrist_2_link: geometry collision cylinder length=0.1 radius=0.04; visual mesh filename=visual/wrist2.stl
- link wrist_3_link: geometry visual mesh filename=visual/wrist3.stl
